Commit message: full and completely rewritten custom ROS package for UR10e + gripper

File: jh_ur10e_hande/urdf/ur10e_hande.urdf.xacro (robot description, xacro)
@@ -7,6 +7,6 @@
   <xacro:include filename="$(find robotiq_description)/urdf/robotiq_hande_gripper.urdf.xacro"/>
   <!-- Attach Hand-E to tool0 -->
-  <xacro:robotiq_hande_gripper parent="tool0">
-    <!-- <origin xyz="0 0 0.01" rpy="0 0 0"/> -->
+  <xacro:robotiq_hande_gripper prefix="" parent="tool0">
+    <origin xyz="0 0 0.01" rpy="0 0 0"/>
   </xacro:robotiq_hande_gripper>
 </robot>

Commit message: save changes

File: jh_ur10e_hande/urdf/ur10e_hande.urdf.xacro (robot description, xacro)
@@ -5,7 +5,10 @@
   <xacro:include filename="$(find robotiq_description)/urdf/robotiq_hande_gripper.urdf.xacro"/>
   <xacro:robotiq_hande_gripper prefix="" parent="tool0">
-    <origin xyz="0 0 0.01" rpy="0 0 0"/>
+    <origin xyz="0 0 0.005" rpy="0 0 0"/>
   </xacro:robotiq_hande_gripper>
   <gazebo>
+    <plugin name="gazebo_ros_control" filename="libgazebo_ros_control.so">
+      <robotNamespace>/</robotNamespace>
+    </plugin>
   </gazebo>
   <gazebo reference="base_link">
